File: Hardware/lanterna_bueno/PCB_led.kicad_sch (KiCad schematic)
At the start: 11 parts, among them J2 Conn_01x02_Male, J3 Conn_01x02_Male, P1 USB_C_Plug_USB2.0, Q2 2SK4075, Q3 2SK4075, Q4 2SK4075, Q5 2SK4075

Commit message: Building
Parts:
- J4, J5, J6, J7: value (none) -> Conn_01x03_Male; footprint (none) -> Connector:3pin 90 pcb solder
Changed lines of the file:
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@@
     (in_bom yes) (on_board yes) (fields_autoplaced)
     (property "Reference" "J7" (id 0) (at 66.675 142.24 0))
-    (property "Value" "" (id 1) (at 66.675 144.78 0))
-    (property "Footprint" "" (id 2) (at 66.04 149.86 0)
+    (property "Value" "Conn_01x03_Male" (id 1) (at 66.675 144.78 0))
+    (property "Footprint" "Connector:3pin 90 pcb solder" (id 2) (at 66.04 149.86 0)
       (effects (font (size 1.27 1.27)) hide)
     )
@@
     (in_bom yes) (on_board yes) (fields_autoplaced)
     (property "Reference" "J5" (id 0) (at 66.675 119.38 0))
-    (property "Value" "" (id 1) (at 66.675 121.92 0))
-    (property "Footprint" "" (id 2) (at 66.04 127 0)
+    (property "Value" "Conn_01x03_Male" (id 1) (at 66.675 121.92 0))
+    (property "Footprint" "Connector:3pin 90 pcb solder" (id 2) (at 66.04 127 0)
       (effects (font (size 1.27 1.27)) hide)
     )
@@
     (in_bom yes) (on_board yes) (fields_autoplaced)
     (property "Reference" "J4" (id 0) (at 66.675 107.95 0))
-    (property "Value" "" (id 1) (at 66.675 110.49 0))
-    (property "Footprint" "" (id 2) (at 66.04 115.57 0)
+    (property "Value" "Conn_01x03_Male" (id 1) (at 66.675 110.49 0))
+    (property "Footprint" "Connector:3pin 90 pcb solder" (id 2) (at 66.04 115.57 0)
       (effects (font (size 1.27 1.27)) hide)
     )
@@
     (in_bom yes) (on_board yes) (fields_autoplaced)
     (property "Reference" "J6" (id 0) (at 66.675 130.81 0))
-    (property "Value" "" (id 1) (at 66.675 133.35 0))
-    (property "Footprint" "" (id 2) (at 66.04 138.43 0)
+    (property "Value" "Conn_01x03_Male" (id 1) (at 66.675 133.35 0))
+    (property "Footprint" "Connector:3pin 90 pcb solder" (id 2) (at 66.04 138.43 0)
       (effects (font (size 1.27 1.27)) hide)
     )
